File: Rev. 1/Eagle/C64_PSU_Combi.brd (EAGLE design)
At the start: 94 x 98 mm, 35 parts, among them J1 0026604050, J2 0026604050, J3 0026604100, J4 0026604040, J5 0026604040, J6 0026604030, J7 10321041

Commit message: Silk Screen Update
Parts:
- added U$31: OPEN_SOURCE_HW, Logo:OPENHW
Other:
- board text added: "1,5KE12A"
- board text added: "100n"
- board text added: "10n/500V"
- board text added: "1M"
- board text added: "1N5908"
- board text added: "47u/50V"
- board text added: "50R"
- board text added: "B32922C3334M"
- board text added: "BV_UI_304_0153"
- board text added: "P6KE15CA"
- board text added: "TEZ10/D230/9V"
- board text added: "http://github.com/ svenpetersen1965"
